File: ZED-F9P_Converter.sch (KiCad schematic (older format))
At the start: 5 parts, among them J1 Conn_01x14, J2 Conn_01x13, J3 Conn_01x14, J4 Conn_01x13, U1 Ublox_ZED_F9P

Commit message: 線幅0.5mmに変更
Parts:
- removed U1: Ublox_ZED_F9P, f9p:UBLOX_ZED_F9P, symbol f9p:Ublox_ZED_F9P
- added U?: f9p_Ublox_ZED_F9P, symbol ZED-F9P_Converter:f9p_Ublox_ZED_F9P
Changed lines of the file:
@@
 EESchema Schematic File Version 4
-LIBS:F9PDIP-cache
-EELAYER 26 0
+EELAYER 29 0
 EELAYER END
 $Descr A4 11693 8268
@@
 $EndDescr
 $Comp
-L f9p:Ublox_ZED_F9P U1
-U 1 1 5E889DF9
-P 5750 3150
-F 0 "U1" H 6091 4775 50  0000 C CNN
-F 1 "Ublox_ZED_F9P" H 6091 4684 50  0000 C CNN
-F 2 "f9p:UBLOX_ZED_F9P" H 5750 3150 50  0001 C CNN
-F 3 "" H 5750 3150 50  0001 C CNN
-	1    5750 3150
-	1    0    0    -1
-$EndComp
-$Comp
 L Connector_Generic:Conn_01x14 J1
 U 1 1 5E88A845
@@
 	7400 4450 6900 4450
 Wire Wire Line
-	4550 4450 4100 4450
-Wire Wire Line
-	4100 4350 4550 4350
-Wire Wire Line
-	4550 4250 4100 4250
-Wire Wire Line
-	4550 4050 4100 4050
-Wire Wire Line
-	4100 4150 4550 4150
-Wire Wire Line
-	4550 3950 4100 3950
-Wire Wire Line
-	4100 3850 4550 3850
-Wire Wire Line
-	4550 3750 4100 3750
-Wire Wire Line
-	4100 3650 4550 3650
-Wire Wire Line
-	4550 3550 4100 3550
-Wire Wire Line
-	4100 3450 4550 3450
-Wire Wire Line
-	4550 3350 4100 3350
-Wire Wire Line
-	4100 3250 4550 3250
-Wire Wire Line
-	4550 2950 4100 2950
-Wire Wire Line
-	4550 1850 4100 1850
-Wire Wire Line
-	4550 2050 4100 2050
-Wire Wire Line
-	4100 2150 4550 2150
-Wire Wire Line
-	4550 2250 4100 2250
-Wire Wire Line
-	4100 2350 4550 2350
-Wire Wire Line
-	4550 2450 4100 2450
-Wire Wire Line
-	4100 2550 4550 2550
-Wire Wire Line
-	4550 2650 4100 2650
-Wire Wire Line
-	4100 2750 4550 2750
-Wire Wire Line
 	5650 5100 5650 4850
 Wire Wire Line
@@
 Connection ~ 4450 3050
 Wire Wire Line
-	4450 3050 4550 3050
-Wire Wire Line
 	4350 2850 4350 5100
 Connection ~ 4350 2850
 Wire Wire Line
-	4350 2850 4550 2850
-Wire Wire Line
 	4250 1950 4250 5100
 Connection ~ 4250 1950
 Wire Wire Line
-	4250 1950 4550 1950
-Wire Wire Line
 	4150 1750 4150 5100
 Connection ~ 4150 1750
-Wire Wire Line
-	4150 1750 4550 1750
 $Comp
 L power:GND #PWR0101
@@
 	1    0    0    -1
 $EndComp
+$Comp
+L ZED-F9P_Converter:f9p_Ublox_ZED_F9P U?
+U 1 1 5E8B41E0
+P 5750 3150
+F 0 "U?" H 6090 4775 50  0000 C CNN
+F 1 "f9p_Ublox_ZED_F9P" H 6090 4684 50  0000 C CNN
+F 2 "" H 5750 3150 50  0001 C CNN
+F 3 "" H 5750 3150 50  0001 C CNN
+	1    5750 3150
+	1    0    0    -1
+$EndComp
+Wire Wire Line
+	4100 4450 4550 4450
+Wire Wire Line
+	4100 4350 4550 4350
+Wire Wire Line
+	4100 4250 4550 4250
+Wire Wire Line
+	4100 4050 4550 4050
+Wire Wire Line
+	4100 4150 4550 4150
+Wire Wire Line
+	4100 3950 4550 3950
+Wire Wire Line
+	4100 3850 4550 3850
+Wire Wire Line
+	4100 3750 4550 3750
+Wire Wire Line
+	4100 3650 4550 3650
+Wire Wire Line
+	4100 3550 4550 3550
+Wire Wire Line
+	4100 3450 4550 3450
+Wire Wire Line
+	4100 3350 4550 3350
+Wire Wire Line
+	4100 3250 4550 3250
+Wire Wire Line
+	4100 2950 4550 2950
+Wire Wire Line
+	4100 1850 4550 1850
+Wire Wire Line
+	4100 2050 4550 2050
+Wire Wire Line
+	4100 2150 4550 2150
+Wire Wire Line
+	4100 2250 4550 2250
+Wire Wire Line
+	4100 2350 4550 2350
+Wire Wire Line
+	4100 2450 4550 2450
+Wire Wire Line
+	4100 2550 4550 2550
+Wire Wire Line
+	4100 2650 4550 2650
+Wire Wire Line
+	4100 2750 4550 2750
+Wire Wire Line
+	4450 3050 4550 3050
+Wire Wire Line
+	4350 2850 4550 2850
+Wire Wire Line
+	4250 1950 4550 1950
+Wire Wire Line
+	4150 1750 4550 1750
 $EndSCHEMATC

Commit message: 軽微な変更
Parts:
- U?: symbol ZED-F9P_Converter:f9p_Ublox_ZED_F9P -> ZED-F9P_Converter-rescue:f9p_Ublox_ZED_F9P-ZED-F9P_Converter
Changed lines of the file:
@@
 EESchema Schematic File Version 4
-EELAYER 29 0
+LIBS:ZED-F9P_Converter-cache
+EELAYER 26 0
 EELAYER END
 $Descr A4 11693 8268
@@
 Date "2020-04-05"
 Rev "1.0"
-Comp "Akinobu Kobayashi"
-Comment1 "Kanazawa Institute of Technology"
+Comp "Mechatroman"
+Comment1 ""
 Comment2 ""
 Comment3 ""
@@
 $EndComp
 $Comp
-L ZED-F9P_Converter:f9p_Ublox_ZED_F9P U?
+L ZED-F9P_Converter-rescue:f9p_Ublox_ZED_F9P-ZED-F9P_Converter U?
 U 1 1 5E8B41E0
 P 5750 3150
